Commit message: update bug

File: Ros_code/mobile_manipulator_body/urdf/robot_base.urdf (robot description, URDF)
Before this commit: robot robot_base, 5 links, 4 joints
Joints:
- removed joint CASTER
- removed joint Lidar
- added joint CASTER_joint: type fixed, parent base_link, child CASTER, origin xyz=0.0759035293244633 1.04273562376855E-05 -0.0299999999999997 rpy=0 0 0, axis 0 0 0
- added joint Lidar_joint: type fixed, parent base_link, child Lidar, origin xyz=0.0659038792794608 1.07773112351106E-05 0.134299800000001 rpy=0 0 0, axis 0 0 0

Commit message: change base_link on urdf code

File: Ros_code/mobile_manipulator_body/urdf/robot_base.urdf (robot description, URDF)
Before this commit: robot robot_base, 5 links, 4 joints
Links:
- added link dummy_link; visual sphere radius=0.001
Joints:
- added joint base_to_dummy: type fixed, parent dummy_link, child base_link, origin xyz=0 0 0 rpy=0 0 0
