Commit message: update ros_code

File: catkin_ws/src/mobile_manipulator_body/urdf/robot_base.urdf.xacro (robot description, xacro)
@@ -13,4 +13,11 @@
   <xacro:include filename="$(find mobile_manipulator_body)/urdf/robot_base.gazebo" />
   <xacro:property name="mesh_path" value="package://mobile_manipulator_body/meshes/" />
+  <!-- base_footprint -->
+  <link name="base_footprint"/>
+  <joint name="base_joint" type="fixed">
+    <parent link="base_footprint"/>
+    <child link="base_link"/>
+    <origin xyz="0 0 0.1" rpy="0 0 0"/>
+  </joint>
   <!-- Base link -->
   <link name="base_link">
